Commit message: feat!: added launch files for instantiating URDF in gazebo

File: urdf_dummy/description/dummy_bot.urdf (robot description, URDF)
Before this commit: robot origins, 2 links, 1 joints
Links:
- removed link base_link
- removed link right_leg
- added link link, mass 1; visual sphere radius=1.0
Joints:
- removed joint base_to_right_leg

Commit message: feat: added base model for robot

File: urdf_dummy/description/dummy_bot.urdf (robot description, URDF)
Before this commit: robot dummy_bot, 1 links, 0 joints
Links:
- removed link link
- added link chassis, mass 1; visual box size=1.0 0.7 0.5
- added link left_wheel, mass 1; visual cylinder length=0.3 radius=0.2
- added link right_wheel, mass 1; visual cylinder length=0.3 radius=0.2
Joints:
- added joint chassis_to_left_wheel: type revolute, parent chassis, child left_wheel, axis 0 1 0, limit lower=-1.79769e+308 upper=1.79769e+308 effort=1000.0 velocity=0.5
- added joint chassis_to_right_wheel: type fixed, parent chassis, child right_wheel, axis 0 1 0, limit lower=-1.79769e+308 upper=1.79769e+308 effort=1000.0 velocity=0.5

Commit message: feat!: added diffDrive plugin

File: urdf_dummy/description/dummy_bot.urdf (robot description, URDF)
Before this commit: robot dummy_bot, 3 links, 2 joints
Links:
- added link back_left_dummy_wheel, mass 1; collision sphere radius=0.2; visual sphere radius=0.2
- added link back_right_dummy_wheel, mass 1; collision sphere radius=0.2; visual sphere radius=0.2
- added link front_left_dummy_wheel, mass 1; collision sphere radius=0.2; visual sphere radius=0.2
- added link front_right_dummy_wheel, mass 1; collision sphere radius=0.2; visual sphere radius=0.2
- added link world
- link chassis: geometry collision box size=1.5 1.0 0.5; visual box size=1.5 1.0 0.5
- link left_wheel: geometry collision cylinder length=0.3 radius=0.2; visual cylinder length=0.3 radius=0.2
- link right_wheel: geometry collision cylinder length=0.3 radius=0.2; visual cylinder length=0.3 radius=0.2
Joints:
- added joint chassis_to_back_left_dummy_wheel: type continuous, parent chassis, child back_left_dummy_wheel
- added joint chassis_to_back_right_dummy_wheel: type continuous, parent chassis, child back_right_dummy_wheel
- added joint chassis_to_front_left_dummy_wheel: type continuous, parent chassis, child front_left_dummy_wheel
- added joint chassis_to_front_right_dummy_wheel: type continuous, parent chassis, child front_right_dummy_wheel
- added joint chassis_to_joint: type fixed, parent world, child chassis, origin xyz=1.5 1.0 0 rpy=0 0 0
- joint chassis_to_right_wheel: type fixed -> revolute

Commit message: fix: physics with urdf model

File: urdf_dummy/description/dummy_bot.urdf (robot description, URDF)
Before this commit: robot dummy_bot, 8 links, 7 joints
Links:
- removed link back_right_dummy_wheel
- removed link chassis
- removed link front_left_dummy_wheel
- removed link front_right_dummy_wheel
- removed link left_wheel
- removed link right_wheel
- removed link world
- added link block, mass 1; collision box size=1.5 1.0 0.5; visual box size=1.5 1.0 0.5
Joints:
- removed joint chassis_to_back_right_dummy_wheel
- removed joint chassis_to_front_left_dummy_wheel
- removed joint chassis_to_front_right_dummy_wheel
- removed joint chassis_to_joint
- removed joint chassis_to_left_wheel
- removed joint chassis_to_right_wheel
- joint chassis_to_back_left_dummy_wheel: parent chassis -> block

Commit message: fix: physics of  urdf model

File: urdf_dummy/description/dummy_bot.urdf (robot description, URDF)
Before this commit: robot dummy_bot, 2 links, 1 joints
Links:
- removed link block
- added link back_right_dummy_wheel, mass 1; collision sphere radius=0.2; visual sphere radius=0.2
- added link chassis, mass 1; collision box size=1.5 1.0 0.5; visual box size=1.5 1.0 0.5
- added link front_left_dummy_wheel, mass 1; collision sphere radius=0.2; visual sphere radius=0.2
- added link front_right_dummy_wheel, mass 1; collision sphere radius=0.2; visual sphere radius=0.2
- added link left_wheel, mass 1; collision cylinder length=0.3 radius=0.2; visual cylinder length=0.3 radius=0.2
- added link right_wheel, mass 1; collision cylinder length=0.3 radius=0.2; visual cylinder length=0.3 radius=0.2
Joints:
- added joint chassis_to_back_right_dummy_wheel: type continuous, parent chassis, child back_right_dummy_wheel, origin xyz=-0.6 -0.25 -0.3 rpy=0 0 0
- added joint chassis_to_front_left_dummy_wheel: type continuous, parent chassis, child front_left_dummy_wheel, origin xyz=0.6 0.25 -0.3 rpy=0 0 0
- added joint chassis_to_front_right_dummy_wheel: type continuous, parent chassis, child front_right_dummy_wheel, origin xyz=0.6 -0.25 -0.3 rpy=0 0 0
- added joint chassis_to_left_wheel: type revolute, parent chassis, child left_wheel, origin xyz=0 0.65 -0.3 rpy=1.57075 0 0, axis 0 1 0, limit lower=-1.79769e+308 upper=1.79769e+308 effort=1000.0 velocity=0.5
- added joint chassis_to_right_wheel: type revolute, parent chassis, child right_wheel, origin xyz=0 -0.65 -0.3 rpy=-1.57075 0 0, axis 0 1 0, limit lower=-1.79769e+308 upper=1.79769e+308 effort=1000.0 velocity=0.5
- joint chassis_to_back_left_dummy_wheel: origin (none) -> xyz=-0.6 0.25 -0.3 rpy=0 0 0; parent block -> chassis

Commit message: feat: add lidar model

File: urdf_dummy/description/dummy_bot.urdf (robot description, URDF)
Before this commit: robot dummy_bot, 7 links, 6 joints
Links:
- added link lidar, mass 0.1; collision cylinder length=0.06 radius=0.09; visual cylinder length=0.06 radius=0.09
Joints:
- added joint chassis_to_lidar: type fixed, parent chassis, child lidar, origin xyz=0 0 0.27 rpy=0 0 0

Commit message: feat!: add abillity to move robot

File: urdf_dummy/description/dummy_bot.urdf (robot description, URDF)
Before this commit: robot dummy_bot, 8 links, 7 joints
Joints:
- joint chassis_to_left_wheel: axis 0 1 0 -> 0 0 1; limit lower=-1.79769e+308 upper=1.79769e+308 effort=1000.0 velocity=0.5 -> lower=-1.79769e+308 upper=1.79769e+308 effort=1000.0 velocity=1.0
- joint chassis_to_right_wheel: axis 0 1 0 -> 0 0 1; limit lower=-1.79769e+308 upper=1.79769e+308 effort=1000.0 velocity=0.5 -> lower=-1.79769e+308 upper=1.79769e+308 effort=1000.0 velocity=1.0; origin xyz=0 -0.65 -0.3 rpy=-1.57075 0 0 -> xyz=0 -0.65 -0.3 rpy=1.57075 0 0

Commit message: feat!: add cameras and tf static

File: urdf_dummy/description/dummy_bot.urdf (robot description, URDF)
Before this commit: robot dummy_bot, 8 links, 7 joints
Links:
- added link camera_back_link, mass 0.001; collision box size=0.01 0.01 0.01; visual box size=0.01 0.01 0.01
- added link camera_front_link, mass 0.001; collision box size=0.01 0.01 0.01; visual box size=0.01 0.01 0.01
- added link camera_left_link, mass 0.001; collision box size=0.01 0.01 0.01; visual box size=0.01 0.01 0.01
- added link camera_right_link, mass 0.001; collision box size=0.01 0.01 0.01; visual box size=0.01 0.01 0.01
Joints:
- added joint camera_back_joint: type fixed, parent chassis, child camera_back_link, origin xyz=-0.77 0 0 rpy=0 0 3.1415
- added joint camera_front_joint: type fixed, parent chassis, child camera_front_link, origin xyz=0.77 0 0 rpy=0 0 0
- added joint camera_left_joint: type fixed, parent chassis, child camera_left_link, origin xyz=0 0.52 0 rpy=0 0 1.57075
- added joint camera_right_joint: type fixed, parent chassis, child camera_right_link, origin xyz=0 -0.52 0 rpy=0 0 -1.57075

Commit message: chour: continius joint remove

File: urdf_dummy/description/dummy_bot.urdf (robot description, URDF)
Before this commit: robot dummy_bot, 12 links, 11 joints
Joints:
- joint chassis_to_back_left_dummy_wheel: type continuous -> fixed
- joint chassis_to_back_right_dummy_wheel: type continuous -> fixed
- joint chassis_to_front_left_dummy_wheel: type continuous -> fixed
- joint chassis_to_front_right_dummy_wheel: type continuous -> fixed
