Commit message: feat!: added actual robot model topics renaming actors

File: urdf_dummy/description/overlord100.urdf (robot description, URDF)
Before this commit: robot overlord100, 12 links, 11 joints
Links:
- removed link camera_back_link
- removed link camera_front_link
- removed link camera_left_link
- removed link camera_right_link
- removed link lidar
- added link lidar_back, mass 0.1; collision box size=0.061 0.041 0.055; visual mesh filename=model://back_lidar.dae
- added link lidar_front, mass 0.1; collision box size=0.061 0.041 0.055; visual mesh filename=model://front_lidar.dae
- added link realsense, mass 0.1; collision box size=0.061 0.041 0.055; visual mesh filename=model://realsense.dae
- added link sonar1, mass 0.1; collision box size=0.061 0.041 0.055; visual mesh filename=model://sonar1.dae
- added link sonar2, mass 0.1; collision box size=0.061 0.041 0.055; visual mesh filename=model://sonar2.dae
- added link sonar3, mass 0.1; collision box size=0.061 0.041 0.055; visual mesh filename=model://sonar3.dae
- added link sonar4, mass 0.1; collision box size=0.061 0.041 0.055; visual mesh filename=model://sonar4.dae
- added link sonar5, mass 0.1; collision box size=0.061 0.041 0.055; visual mesh filename=model://sonar5.dae
- added link sonar6, mass 0.1; collision box size=0.061 0.041 0.055; visual mesh filename=model://sonar6.dae
- added link sonar7, mass 0.1; collision box size=0.061 0.041 0.055; visual mesh filename=model://sonar7.dae
- added link sonar8, mass 0.1; collision box size=0.061 0.041 0.055; visual mesh filename=model://sonar8.dae
- link back_left_dummy_wheel: geometry collision sphere radius=0.07; visual mesh filename=model://back_left_wheel.dae
- link back_right_dummy_wheel: geometry collision sphere radius=0.07; visual mesh filename=model://back_right_wheel.dae
- link chassis: mass 1 -> 60.5; geometry collision box size=0.67 0.93 0.2; visual mesh filename=model://base.dae
- link front_left_dummy_wheel: geometry collision sphere radius=0.07; visual mesh filename=model://front_left_wheel.dae
- link front_right_dummy_wheel: geometry collision sphere radius=0.07; visual mesh filename=model://front_right_wheel.dae
- link left_wheel: geometry collision cylinder length=0.06 radius=0.07; visual mesh filename=model://left_wheel.dae
- link right_wheel: geometry collision cylinder length=0.06 radius=0.07; visual mesh filename=model://right_wheel.dae
Joints:
- removed joint camera_back_joint
- removed joint camera_front_joint
- removed joint camera_left_joint
- removed joint camera_right_joint
- removed joint chassis_to_lidar
- added joint chassis_to_lidar_back: type fixed, parent chassis, child lidar_back, origin xyz=-0.26 -0.42 0 rpy=0 0 0
- added joint chassis_to_lidar_front: type fixed, parent chassis, child lidar_front, origin xyz=0.26 0.43 0 rpy=0 0 0
- added joint chassis_to_realsense: type fixed, parent chassis, child realsense, origin xyz=0 0.48 -0.032
- added joint chassis_to_sonar1: type fixed, parent chassis, child sonar1, origin xyz=0.138 0.45 -0.032
- added joint chassis_to_sonar2: type fixed, parent chassis, child sonar2, origin xyz=-0.138 0.45 -0.032
- added joint chassis_to_sonar3: type fixed, parent chassis, child sonar3, origin xyz=-0.3 0.24 -0.032
- added joint chassis_to_sonar4: type fixed, parent chassis, child sonar4, origin xyz=-0.3 -0.23 -0.032
- added joint chassis_to_sonar5: type fixed, parent chassis, child sonar5, origin xyz=-0.138 -0.45 -0.032
- added joint chassis_to_sonar6: type fixed, parent chassis, child sonar6, origin xyz=0.138 -0.45 -0.032
- added joint chassis_to_sonar7: type fixed, parent chassis, child sonar7, origin xyz=0.3 -0.23 -0.032
- added joint chassis_to_sonar8: type fixed, parent chassis, child sonar8, origin xyz=0.3 0.24 -0.032
- joint chassis_to_back_left_dummy_wheel: origin xyz=-0.6 0.25 -0.3 rpy=0 0 0 -> xyz=0.27 -0.42 -0.15 rpy=0 0 0
- joint chassis_to_back_right_dummy_wheel: origin xyz=-0.6 -0.25 -0.3 rpy=0 0 0 -> xyz=-0.27 -0.42 -0.15 rpy=0 0 0
- joint chassis_to_front_left_dummy_wheel: origin xyz=0.6 0.25 -0.3 rpy=0 0 0 -> xyz=0.23 0.40 -0.15 rpy=0 0 0
- joint chassis_to_front_right_dummy_wheel: origin xyz=0.6 -0.25 -0.3 rpy=0 0 0 -> xyz=-0.23 0.40 -0.15 rpy=0 0 0
- joint chassis_to_left_wheel: axis 0 0 1 -> 1 0 0; limit lower=-1.79769e+308 upper=1.79769e+308 effort=1000.0 velocity=1.0 -> lower=-1.79769e+308 upper=1.79769e+308 effort=1000.0 velocity=10.0; origin xyz=0 0.65 -0.3 rpy=1.57075 0 0 -> xyz=0.33 -0.045 -0.15 rpy=0 0 3.14
- joint chassis_to_right_wheel: axis 0 0 1 -> 1 0 0; limit lower=-1.79769e+308 upper=1.79769e+308 effort=1000.0 velocity=1.0 -> lower=-1.79769e+308 upper=1.79769e+308 effort=1000.0 velocity=10.0; origin xyz=0 -0.65 -0.3 rpy=1.57075 0 0 -> xyz=-0.33 -0.045 -0.15 rpy=0 0 3.14

Commit message: fix: controller for simulation and lidars range

File: urdf_dummy/description/overlord100.urdf (robot description, URDF)
Before this commit: robot overlord100, 18 links, 17 joints
Joints:
- joint chassis_to_left_wheel: limit lower=-1.79769e+308 upper=1.79769e+308 effort=1000.0 velocity=10.0 -> lower=-1.79769e+308 upper=1.79769e+308 effort=1000.0 velocity=100.0
- joint chassis_to_right_wheel: limit lower=-1.79769e+308 upper=1.79769e+308 effort=1000.0 velocity=10.0 -> lower=-1.79769e+308 upper=1.79769e+308 effort=1000.0 velocity=100.0

Commit message: feat:sonars and realsense in rviz

File: urdf_dummy/description/overlord100.urdf (robot description, URDF)
Before this commit: robot overlord100, 18 links, 17 joints
Joints:
- joint chassis_to_sonar1: origin xyz=0.138 0.45 -0.032 -> xyz=0.138 0.45 -0.032 rpy=0 0 1.57075 
- joint chassis_to_sonar2: origin xyz=-0.138 0.45 -0.032 -> xyz=-0.138 0.45 -0.032 rpy=0 0 1.57075
- joint chassis_to_sonar3: origin xyz=-0.3 0.24 -0.032 -> xyz=-0.3 0.24 -0.032 rpy=0 0.5 3.1415
- joint chassis_to_sonar4: origin xyz=-0.3 -0.23 -0.032 -> xyz=-0.3 -0.23 -0.032 rpy=0 0.5 3.1415
- joint chassis_to_sonar5: origin xyz=-0.138 -0.45 -0.032 -> xyz=-0.138 -0.45 -0.032 rpy=0 0 -1.57075
- joint chassis_to_sonar6: origin xyz=0.138 -0.45 -0.032 -> xyz=0.138 -0.45 -0.032 rpy=0 0 -1.57075
- joint chassis_to_sonar7: origin xyz=0.3 -0.23 -0.032 -> xyz=0.3 -0.23 -0.032 rpy=0 0.5 0
- joint chassis_to_sonar8: origin xyz=0.3 0.24 -0.032 -> xyz=0.3 0.24 -0.032 rpy=0 0.5 0

Commit message: fix: single lidar

File: urdf_dummy/description/overlord100.urdf (robot description, URDF)
Before this commit: robot overlord100, 18 links, 17 joints
Links:
- removed link lidar_front
Joints:
- removed joint chassis_to_lidar_front
- joint chassis_to_lidar_back: origin xyz=-0.26 -0.42 0 rpy=0 0 0 -> xyz=0 0 0 rpy=0 0 0

File: urdf_dummy/description/overlord100_with_diffdrive.urdf (robot description, URDF)
Before this commit: robot overlord100, 18 links, 17 joints
Links:
- removed link lidar_front
Joints:
- removed joint chassis_to_lidar_front

Commit message: Sim with map displaying. Slam launches with separate commands

File: urdf_dummy/description/overlord100.urdf (robot description, URDF)
Before this commit: robot overlord100, 17 links, 16 joints
Links:
- added link lidar_front, mass 0.1; collision box size=0.061 0.041 0.055; visual mesh filename=model://front_lidar.dae
- added link lidar_virtual
Joints:
- added joint chassis_to_lidar_front: type fixed, parent chassis, child lidar_front, origin xyz=0.26 0.43 0 rpy=0 0 0
- added joint chassis_to_lidar_virtual: type fixed, parent chassis, child lidar_virtual, origin xyz=0 0 0 rpy=0 0 0
- joint chassis_to_lidar_back: origin xyz=0 0 0 rpy=0 0 0 -> xyz=-0.26 -0.43 0 rpy=0 0 0
